File: Board Versions/70mm by 50mm Ver3.0 esp32-s2/Board Files/KiCad/esp32-s2 with separate heatbed/heatbed_70x50_7R.kicad_pcb (KiCad board)
At the start: 2 copper layers, 87.9 x 60.2 mm, 5 parts

Commit message: Name nets
Connections:
- J** pad 1: (no net) -> heater
- J** pad 2: (no net) -> heater
Routing:
- net heater: track 0.00 -> 5973.9 mm
- net (no net): track 5973.9 -> 0.00 mm
