File: Board Versions/70mm by 50mm Ver3.0 esp32-s2/Board Files/KiCad/esp32-s2 with separate heatbed/heatbed_80x60_1R6.kicad_pcb (KiCad board)
At the start: 2 copper layers, 99.1 x 77.6 mm, 5 parts

Commit message: Add missing caution
Other:
- board text added: "CAUTION"
- board text added: "HOT SURFACE"
Changed lines of the file:
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@@
   )
   (gr_line (start 98.171 154.94) (end 98.171 95.1216) (layer "F.SilkS") (width 1))
+  (gr_arc (start 56.9988 120.6008) (mid 56.580418 119.97415) (end 56.433691 119.235093) (layer "F.SilkS") (width 0.6))
+  (gr_line (start 54.5988 124.6698) (end 62.5988 124.6698) (layer "F.SilkS") (width 0.6))
+  (gr_line (start 50.5988 126.6698) (end 58.5988 112.6698) (layer "F.SilkS") (width 0.6))
+  (gr_arc (start 58.5988 120.6698) (mid 58.180035 120.043074) (end 58.032984 119.3038) (layer "F.SilkS") (width 0.6))
+  (gr_arc (start 60.9988 122.2008) (mid 60.851811 122.939762) (end 60.433223 123.566223) (layer "F.SilkS") (width 0.6))
+  (gr_arc (start 57.7988 122.2008) (mid 57.651811 122.939762) (end 57.233223 123.566223) (layer "F.SilkS") (width 0.6))
+  (gr_arc (start 60.1988 120.6008) (mid 59.780418 119.97415) (end 59.633691 119.235093) (layer "F.SilkS") (width 0.6))
+  (gr_line (start 60.1988 120.6008) (end 60.4328 120.8358) (layer "F.SilkS") (width 0.6))
+  (gr_line (start 58.5988 112.6698) (end 66.5988 126.6698) (layer "F.SilkS") (width 0.6))
+  (gr_arc (start 58.8328 120.9038) (mid 59.251641 121.530144) (end 59.398909 122.269093) (layer "F.SilkS") (width 0.6))
+  (gr_arc (start 60.4328 120.8358) (mid 60.851258 121.462067) (end 60.998202 122.2008) (layer "F.SilkS") (width 0.6))
+  (gr_line (start 58.5988 120.6698) (end 58.8328 120.9038) (layer "F.SilkS") (width 0.6))
+  (gr_arc (start 59.3988 122.2698) (mid 59.251811 123.008762) (end 58.833223 123.635223) (layer "F.SilkS") (width 0.6))
   (gr_line (start 98.171 154.94) (end 17.5632 154.94) (layer "F.SilkS") (width 1))
+  (gr_arc (start 56.4328 119.2358) (mid 56.579865 118.496456) (end 56.99867 117.86967) (layer "F.SilkS") (width 0.6))
+  (gr_arc (start 57.2328 120.8358) (mid 57.651258 121.462067) (end 57.798202 122.2008) (layer "F.SilkS") (width 0.6))
   (gr_line (start 17.5632 95.1216) (end 98.171 95.1216) (layer "F.SilkS") (width 1))
+  (gr_arc (start 59.6328 119.2358) (mid 59.779865 118.496456) (end 60.19867 117.86967) (layer "F.SilkS") (width 0.6))
+  (gr_arc (start 58.0328 119.3038) (mid 58.179865 118.564456) (end 58.59867 117.93767) (layer "F.SilkS") (width 0.6))
+  (gr_line (start 56.9988 120.6008) (end 57.2328 120.8358) (layer "F.SilkS") (width 0.6))
   (gr_line (start 17.5632 95.1216) (end 17.5632 154.94) (layer "F.SilkS") (width 1))
+  (gr_line (start 50.5988 126.6698) (end 66.5988 126.6698) (layer "F.SilkS") (width 0.6))
   (gr_rect (start 17.4632 94.9216) (end 98.044 155.067) (layer "Eco1.User") (width 0.15) (fill none))
   (gr_rect (start 7.62 86.36) (end 106.68 163.957) (layer "Edge.Cuts") (width 0.2) (fill none))
+  (gr_text "CAUTION" (at 58.5988 130.4198) (layer "F.SilkS")
+    (effects (font (size 2.4 2.4) (thickness 0.4)))
+  )
+  (gr_text "HOT SURFACE" (at 58.5988 133.0698) (layer "F.SilkS")
+    (effects (font (size 1.4 1.4) (thickness 0.24)))
+  )
   (gr_text "80mm x 60mm" (at 103.1748 134.366 90) (layer "F.SilkS")
     (effects (font (size 1.6 1.6) (thickness 0.2)) (justify left))

Commit message: Correct resistance for heatbed 1.6
Routing:
- net (no net): track 4008.8 -> 3273.4 mm
Other:
- board text added: "Calculated: 1.56R@20°C"
- board text removed: "Calculated: 1.57R@20°C"

Commit message: Name nets
Connections:
- J** pad 1: (no net) -> heater
- J** pad 2: (no net) -> heater
Routing:
- net heater: track 0.00 -> 3273.4 mm
- net (no net): track 3273.4 -> 0.00 mm

Commit message: Add bottom silk screen
Other:
- board text added: "Calculated: 1.59R@20°C"
- board text added: "Measured:"
- board text removed: "Calculated: 1.56R@20°C"
Changed lines of the file:
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@@
     (pad "" np_thru_hole circle (at 0 16) (size 3.2 3.2) (drill 3.2) (layers F&B.Cu *.Mask))
   )
+  (gr_rect (start 42.58 156.4) (end 57.82 158.94) (layer "B.SilkS") (width 0.12) (fill solid))
   (gr_line (start 98.171 154.94) (end 98.171 95.1216) (layer "F.SilkS") (width 1))
   (gr_arc (start 56.9988 120.6008) (mid 56.580418 119.97415) (end 56.433691 119.235093) (layer "F.SilkS") (width 0.6))
@@
   (gr_rect (start 17.4632 94.9216) (end 98.044 155.067) (layer "Eco1.User") (width 0.15) (fill none))
   (gr_rect (start 7.62 86.36) (end 106.68 163.957) (layer "Edge.Cuts") (width 0.2) (fill none))
+  (gr_text "Calculated: 1.59R@20°C" (at 71.12 154.94) (layer "B.SilkS")
+    (effects (font (size 1.6 1.6) (thickness 0.2)) (justify left mirror))
+  )
+  (gr_text "Measured:" (at 71.12 157.48) (layer "B.SilkS")
+    (effects (font (size 1.6 1.6) (thickness 0.2)) (justify left mirror))
+  )
   (gr_text "CAUTION" (at 58.5988 130.4198) (layer "F.SilkS")
     (effects (font (size 2.4 2.4) (thickness 0.4)))
@@
     (effects (font (size 2.4 2.4) (thickness 0.4)) (justify left))
   )
-  (gr_text "Calculated: 1.56R@20°C" (at 44.8818 159.8168) (layer "F.SilkS")
-    (effects (font (size 1.6 1.6) (thickness 0.2)) (justify left))
-  )
   (segment (start 48.7172 95.6564) (end 48.7172 155.4226) (width 0.98) (layer "F.Cu") (net 1))
